Commit message: Fix drone orientation + attitude stabilization; retrain (99.8% success)
The rendered drone was flying on its side with the gripper pointing sideways:
- root cause: the gripper URDF was authored Y-up while Isaac's world + the env's
  flight model/stabilizer are Z-up, so the body got leveled onto its side.
- fix: re-authored drone_with_gripper.urdf Z-up (rotors horizontal in X-Y, gripper
  hangs straight down -Z); re-converted to USD.
- added attitude stabilization to the env (level the body + damp angular velocity)
  so it flies upright like a real quad instead of free-spinning (yaw didn't affect
  reward, so the old policy just let it spin).
- made the gripper links VISUAL-ONLY (the cube was penetrating the finger collision
  boxes where it magnetically attaches -> ejected grasps + contact-pair OOM).

Retrained on the corrected level drone: deterministic eval EPISODE_SUCCESS_RATE
=99.8%, grasp 90%. Rollout now shows an upright quad with the gripper down,
grasping and delivering the cube. render_rollout.py follow-cam + mac-friendly mp4.

Co-Authored-By: Claude Opus 4.8 (1M context) <noreply@anthropic.com>

File: skyvla_isaac/assets/drone_with_gripper.urdf (robot description, URDF)
Before this commit: robot drone_with_gripper, 10 links, 9 joints
Links:
- removed link boom_z
- removed link rotor_zn
- removed link rotor_zp
- added link boom_y; visual box size=0.025 0.42 0.02
- added link rotor_yn; visual cylinder length=0.012 radius=0.10
- added link rotor_yp; visual cylinder length=0.012 radius=0.10
- link arm: mass 0.02 -> 0.03; geometry visual cylinder length=0.30 radius=0.012
- link base: geometry collision box size=0.14 0.14 0.05; visual box size=0.14 0.14 0.05
- link boom_x: geometry visual box size=0.42 0.025 0.02
- link finger_l: geometry visual box size=0.02 0.05 0.08
- link finger_r: geometry visual box size=0.02 0.05 0.08
- link rotor_xn: geometry visual cylinder length=0.012 radius=0.10
- link rotor_xp: geometry visual cylinder length=0.012 radius=0.10
Joints:
- removed joint j_boom_z
- removed joint j_rzn
- removed joint j_rzp
- added joint j_boom_y: type fixed, parent base, child boom_y, origin xyz=0 0 0.01
- added joint j_ryn: type fixed, parent base, child rotor_yn, origin xyz=0 -0.21 0.03
- added joint j_ryp: type fixed, parent base, child rotor_yp, origin xyz=0 0.21 0.03
- joint grip_l: origin xyz=0.045 -0.31 0 -> xyz=0.05 0 -0.32
- joint grip_r: origin xyz=-0.045 -0.31 0 -> xyz=-0.05 0 -0.32
- joint j_boom_x: origin xyz=0 0 0 -> xyz=0 0 0.01
- joint j_rxn: origin xyz=-0.21 0.03 0 -> xyz=-0.21 0 0.03
- joint j_rxp: origin xyz=0.21 0.03 0 -> xyz=0.21 0 0.03
- joint lower: axis 0 -1 0 -> 0 0 -1; origin xyz=0 -0.03 0 -> xyz=0 0 -0.03

Commit message: Real-physics drone pick-and-place: 4-jaw cage gripper, rigid mount, converged policy
Gripper now grasps via real PhysX contact+friction (no teleport/magnetic hack):
- 4-jaw cage (finger_xl/xr/yl/yr) boxes in a free cube; flat 2-finger pinch ejected it.
- Rigid mount: stiff lower joint (stiffness 8000, effort 200) + realistic base
  inertia (1e-3 -> 1.2e-2/2.2e-2) so the gripper no longer telescopes or flings
  the drone. Verified: arm extension 0.21m -> 0.001m, body stays level under stress.
- Reward balance that converges: strong-but-low-plateau lift gate (60*cube_h, cap
  0.15) for grasp discovery + dominant placement (40*place + 25*carry + 80*success)
  gated on a real grasp; curriculum_p 0.7.

Eval (512 episodes, deterministic): grasp 70.4%, deliver 68.5%, full pick-and-place
episode success 71.7%.

Co-Authored-By: Claude Opus 4.8 <noreply@anthropic.com>

File: skyvla_isaac/assets/drone_with_gripper.urdf (robot description, URDF)
Before this commit: robot drone_with_gripper, 10 links, 9 joints
Links:
- removed link finger_l
- removed link finger_r
- added link finger_xl, mass 0.02; collision box size=0.012 0.07 0.05; visual box size=0.012 0.07 0.05
- added link finger_xr, mass 0.02; collision box size=0.012 0.07 0.05; visual box size=0.012 0.07 0.05
- added link finger_yl, mass 0.02; collision box size=0.07 0.012 0.05; visual box size=0.07 0.012 0.05
- added link finger_yr, mass 0.02; collision box size=0.07 0.012 0.05; visual box size=0.07 0.012 0.05
- link base: mass 0.35 -> 1.5
Joints:
- removed joint grip_l
- removed joint grip_r
- added joint grip_xl: type prismatic, parent arm, child finger_xl, origin xyz=0.04 0 -0.30, axis -1 0 0, limit lower=0.0 upper=0.02 effort=40 velocity=1.0
- added joint grip_xr: type prismatic, parent arm, child finger_xr, origin xyz=-0.04 0 -0.30, axis 1 0 0, limit lower=0.0 upper=0.02 effort=40 velocity=1.0
- added joint grip_yl: type prismatic, parent arm, child finger_yl, origin xyz=0 0.04 -0.30, axis 0 -1 0, limit lower=0.0 upper=0.02 effort=40 velocity=1.0
- added joint grip_yr: type prismatic, parent arm, child finger_yr, origin xyz=0 -0.04 -0.30, axis 0 1 0, limit lower=0.0 upper=0.02 effort=40 velocity=1.0
